Commit message: Lots of Work Done!

File: Desktop/catkin_ws_dos/src/hw2/planar_robot.urdf (robot description, URDF)
Before this commit: robot planar_robot, 2 links, 2 joints
Links:
- added link base_link; visual cylinder length=0.6 radius=0.2
- link link1: geometry visual box size=1 0.5 0.2
- link link2: geometry visual box size=1 0.5 0.2
Joints:
- joint joint1: child link2 -> link1; parent link1 -> base_link
- joint joint2: origin xyz=1 1 0 rpy=0 0 0 -> xyz=0 0 0 rpy=0 0 0
