Commit message: Transformer works URDF kind of works

File: planar_robot.urdf (robot description, URDF)
Before this commit: robot planar_robot, 3 links, 2 joints
Joints:
- joint joint2: origin xyz=0 0 0 rpy=0 0 0 -> xyz=1 0 0 rpy=0 0 0

Commit message: Added end link for marker

File: planar_robot.urdf (robot description, URDF)
Before this commit: robot planar_robot, 3 links, 2 joints
Links:
- added link link3; visual cylinder length=0.1 radius=0.1
Joints:
- added joint joint3: type fixed, parent link2, child link3, origin xyz=1 0 0 rpy=0 0 0, axis 0 0 1
